Commit message: feat: implement minimal simulation rebuild based on best practices (EKF + bridge.yaml)

File: src/khr2026_team1_simulation/urdf/robot.urdf.xacro (robot description, xacro)
@@ -1,4 +1,7 @@
 <?xml version="1.0"?>
 <robot name="khr2026_robot" xmlns:xacro="http://www.ros.org/wiki/xacro">
+   <material name="blue"><color rgba="0.0 0.0 0.8 1.0"/></material>
+   <material name="black"><color rgba="0.1 0.1 0.1 1.0"/></material>
+   <material name="grey"><color rgba="0.5 0.5 0.5 1.0"/></material>
   <xacro:include filename="$(find khr2026_team1_simulation)/urdf/mecanum_wheel.xacro"/>
   <xacro:include filename="$(find khr2026_team1_simulation)/urdf/camera.xacro"/>
@@ -6,36 +9,68 @@
   <xacro:include filename="$(find khr2026_team1_simulation)/urdf/lidar.xacro"/>
   <xacro:robot_lidar parent_link="base_link"/>
-  <xacro:property name="wheel_radius" value="0.05"/><xacro:property name="wheel_width" value="0.04"/>
-  <xacro:property name="base_width" value="0.4"/><xacro:property name="base_length" value="0.5"/><xacro:property name="base_height" value="0.1"/>
-  <link name="base_footprint"/>
-  <joint name="base_joint" type="fixed">
-    <parent link="base_footprint"/>
-    <child link="base_link"/>
-    <origin xyz="0 0 0" rpy="0 0 0"/>
-  </joint>
-  <link name="base_link">
-    <visual><origin xyz="0 0 ${base_height/2}"/><geometry><box size="${base_length} ${base_width} ${base_height}"/></geometry><material name="blue"><color rgba="0.0 0.0 0.8 1.0"/></material></visual>
-    <collision><origin xyz="0 0 ${base_height/2}"/><geometry><box size="${base_length} ${base_width} ${base_height}"/></geometry></collision>
-    <inertial><origin xyz="0 0 ${base_height/2}"/><mass value="10.0"/><inertia ixx="0.1" ixy="0" ixz="0" iyy="0.1" iyz="0" izz="0.1"/></inertial>
-  </link>
-  <xacro:robot_camera base_height="${base_height}"/>
-  <xacro:robot_hand base_link="base_link" base_length="${base_length}" base_width="${base_width}" base_height="${base_height}"/>
-  <xacro:mecanum_wheel prefix="front_left" side="1" radius="${wheel_radius}" width="${wheel_width}" x="0.1725" y="0.2425" z="-0.02"/>
-  <xacro:mecanum_wheel prefix="front_right" side="-1" radius="${wheel_radius}" width="${wheel_width}" x="0.1725" y="-0.2425" z="-0.02"/>
-  <xacro:mecanum_wheel prefix="rear_left" side="1" radius="${wheel_radius}" width="${wheel_width}" x="-0.1725" y="0.2425" z="-0.02"/>
-  <xacro:mecanum_wheel prefix="rear_right" side="-1" radius="${wheel_radius}" width="${wheel_width}" x="-0.1725" y="-0.2425" z="-0.02"/>
-  <gazebo>
-    <plugin filename="gz-sim-mecanum-drive-system" name="gz::sim::systems::MecanumDrive">
-      <front_left_joint>front_left_wheel_joint</front_left_joint>
-      <front_right_joint>front_right_wheel_joint</front_right_joint>
-      <back_left_joint>rear_left_wheel_joint</back_left_joint>
-      <back_right_joint>rear_right_wheel_joint</back_right_joint>
-      <wheel_separation>0.485</wheel_separation>
-      <wheelbase>0.345</wheelbase>
-      <wheel_radius>${wheel_radius}</wheel_radius>
-      <odom_publish_frequency>50</odom_publish_frequency>
-      <frame_id>odom</frame_id>
-      <child_frame_id>base_link</child_frame_id>
-    </plugin>
-  </gazebo>
+   <xacro:property name="wheel_radius" value="0.05"/><xacro:property name="wheel_width" value="0.04"/>
+   <xacro:property name="base_width" value="0.4"/><xacro:property name="base_length" value="0.5"/><xacro:property name="base_height" value="0.1"/>
+   <link name="base_footprint"/>
+   <joint name="base_joint" type="fixed">
+     <parent link="base_footprint"/>
+     <child link="base_link"/>
+     <origin xyz="0 0 0.07" rpy="0 0 0"/>
+   </joint>
+   <link name="base_link">
+     <visual><origin xyz="0 0 0"/><geometry><box size="${base_length} ${base_width} ${base_height}"/></geometry><material name="blue"/></visual>
+     <collision><origin xyz="0 0 0"/><geometry><box size="${base_length} ${base_width} ${base_height}"/></geometry></collision>
+     <inertial><origin xyz="0 0 0"/><mass value="10.0"/><inertia ixx="0.1" ixy="0" ixz="0" iyy="0.1" iyz="0" izz="0.1"/></inertial>
+   </link>
+   <gazebo reference="base_link">
+     <material>Gazebo/Blue</material>
+   </gazebo>
+   <xacro:robot_camera base_height="${base_height}"/>
+   <xacro:robot_hand base_link="base_link" base_length="${base_length}" base_width="${base_width}" base_height="${base_height}"/>
+   <xacro:mecanum_wheel prefix="front_left" side="1" radius="${wheel_radius}" width="${wheel_width}" x="0.1725" y="0.2425" z="-0.02"/>
+   <xacro:mecanum_wheel prefix="front_right" side="-1" radius="${wheel_radius}" width="${wheel_width}" x="0.1725" y="-0.2425" z="-0.02"/>
+   <xacro:mecanum_wheel prefix="rear_left" side="1" radius="${wheel_radius}" width="${wheel_width}" x="-0.1725" y="0.2425" z="-0.02"/>
+   <xacro:mecanum_wheel prefix="rear_right" side="-1" radius="${wheel_radius}" width="${wheel_width}" x="-0.1725" y="-0.2425" z="-0.02"/>
+   <gazebo>
+     <plugin filename="gz-sim-mecanum-drive-system" name="gz::sim::systems::MecanumDrive">
+       <front_left_joint>front_left_wheel_joint</front_left_joint>
+       <front_right_joint>front_right_wheel_joint</front_right_joint>
+       <back_left_joint>rear_left_wheel_joint</back_left_joint>
+       <back_right_joint>rear_right_wheel_joint</back_right_joint>
+       <wheel_separation>0.485</wheel_separation>
+       <wheelbase>0.345</wheelbase>
+       <wheel_radius>${wheel_radius}</wheel_radius>
+       <topic>/model/khr2026_robot/cmd_vel</topic>
+       <odom_topic>/model/khr2026_robot/odometry</odom_topic>
+       <tf_topic>/model/khr2026_robot/tf</tf_topic>
+       <frame_id>odom</frame_id>
+       <child_frame_id>base_footprint</child_frame_id>
+       <robot_base_frame>base_footprint</robot_base_frame>
+       <footprint_frame_id>base_footprint</footprint_frame_id>
+       <publish_odom_tf>false</publish_odom_tf>
+       <publish_wheel_tf>false</publish_wheel_tf>
+     </plugin>
+     <plugin filename="gz-sim-joint-state-publisher-system" name="gz::sim::systems::JointStatePublisher">
+       <topic>/world/khr2026_field_generated/model/khr2026_robot/joint_state</topic>
+       <joint_name>front_left_wheel_joint</joint_name>
+       <joint_name>front_right_wheel_joint</joint_name>
+       <joint_name>rear_left_wheel_joint</joint_name>
+       <joint_name>rear_right_wheel_joint</joint_name>
+     </plugin>
+     <plugin filename="gz-sim-imu-system" name="gz::sim::systems::Imu">
+     </plugin>
+   </gazebo>
+   <link name="imu_link">
+     <inertial><mass value="0.01"/><inertia ixx="1e-5" ixy="0" ixz="0" iyy="1e-5" iyz="0" izz="1e-5"/></inertial>
+   </link>
+   <joint name="imu_joint" type="fixed">
+     <parent link="base_link"/><child link="imu_link"/><origin xyz="0 0 0.05"/>
+   </joint>
+   <gazebo reference="imu_link">
+     <sensor name="imu_sensor" type="imu">
+       <always_on>1</always_on>
+       <update_rate>100</update_rate>
+       <visualize>true</visualize>
+       <topic>imu</topic>
+     </sensor>
+   </gazebo>
 </robot>
