Commit message: Add usage instructions for simulation/real mode and related launch changes

File: src/khr2026_team1_simulation/urdf/hand.xacro (robot description, xacro)
@@ -5,5 +5,5 @@
       <visual><origin xyz="0 0 0.15"/><geometry><box size="0.05 0.2 0.3"/></geometry><material name="grey"><color rgba="0.5 0.5 0.5 1.0"/></material></visual>
       <collision><origin xyz="0 0 0.15"/><geometry><box size="0.05 0.2 0.3"/></geometry></collision>
-      <inertial><mass value="1.0"/><inertia ixx="0.01" iyy="0.01" izz="0.01"/></inertial>
+      <inertial><mass value="1.0"/><inertia ixx="0.01" ixy="0" ixz="0" iyy="0.01" iyz="0" izz="0.01"/></inertial>
     </link>
     <joint name="lift_joint" type="prismatic">
@@ -13,5 +13,5 @@
       <visual><geometry><box size="0.1 0.2 0.05"/></geometry></visual>
       <collision><geometry><box size="0.1 0.2 0.05"/></geometry></collision>
-      <inertial><mass value="0.2"/><inertia ixx="0.001" iyy="0.001" izz="0.001"/></inertial>
+      <inertial><mass value="0.2"/><inertia ixx="0.001" ixy="0" ixz="0" iyy="0.001" iyz="0" izz="0.001"/></inertial>
     </link>
     <joint name="gripper_base_joint" type="fixed">
@@ -21,5 +21,5 @@
       <visual><origin xyz="0.05 0 0"/><geometry><box size="0.1 0.02 0.05"/></geometry></visual>
       <collision><origin xyz="0.05 0 0"/><geometry><box size="0.1 0.02 0.05"/></geometry></collision>
-      <inertial><mass value="0.1"/><inertia ixx="0.0001" iyy="0.0001" izz="0.0001"/></inertial>
+      <inertial><mass value="0.1"/><inertia ixx="0.0001" ixy="0" ixz="0" iyy="0.0001" iyz="0" izz="0.0001"/></inertial>
     </link>
     <joint name="left_finger_joint" type="revolute">
@@ -29,5 +29,5 @@
       <visual><origin xyz="0.05 0 0"/><geometry><box size="0.1 0.02 0.05"/></geometry></visual>
       <collision><origin xyz="0.05 0 0"/><geometry><box size="0.1 0.02 0.05"/></geometry></collision>
-      <inertial><mass value="0.1"/><inertia ixx="0.0001" iyy="0.0001" izz="0.0001"/></inertial>
+      <inertial><mass value="0.1"/><inertia ixx="0.0001" ixy="0" ixz="0" iyy="0.0001" iyz="0" izz="0.0001"/></inertial>
     </link>
     <joint name="right_finger_joint" type="revolute">

File: src/khr2026_team1_simulation/urdf/robot.urdf.xacro (robot description, xacro)
@@ -4,10 +4,18 @@
   <xacro:include filename="$(find khr2026_team1_simulation)/urdf/camera.xacro"/>
   <xacro:include filename="$(find khr2026_team1_simulation)/urdf/hand.xacro"/>
+  <xacro:include filename="$(find khr2026_team1_simulation)/urdf/lidar.xacro"/>
+  <xacro:robot_lidar parent_link="base_link"/>
   <xacro:property name="wheel_radius" value="0.05"/><xacro:property name="wheel_width" value="0.04"/>
   <xacro:property name="base_width" value="0.4"/><xacro:property name="base_length" value="0.5"/><xacro:property name="base_height" value="0.1"/>
+  <link name="base_footprint"/>
+  <joint name="base_joint" type="fixed">
+    <parent link="base_footprint"/>
+    <child link="base_link"/>
+    <origin xyz="0 0 0" rpy="0 0 0"/>
+  </joint>
   <link name="base_link">
     <visual><origin xyz="0 0 ${base_height/2}"/><geometry><box size="${base_length} ${base_width} ${base_height}"/></geometry><material name="blue"><color rgba="0.0 0.0 0.8 1.0"/></material></visual>
     <collision><origin xyz="0 0 ${base_height/2}"/><geometry><box size="${base_length} ${base_width} ${base_height}"/></geometry></collision>
-    <inertial><origin xyz="0 0 ${base_height/2}"/><mass value="10.0"/><inertia ixx="0.1" iyy="0.1" izz="0.1"/></inertial>
+    <inertial><origin xyz="0 0 ${base_height/2}"/><mass value="10.0"/><inertia ixx="0.1" ixy="0" ixz="0" iyy="0.1" iyz="0" izz="0.1"/></inertial>
   </link>
   <xacro:robot_camera base_height="${base_height}"/>
@@ -18,7 +26,15 @@
   <xacro:mecanum_wheel prefix="rear_right" side="-1" radius="${wheel_radius}" width="${wheel_width}" x="-0.1725" y="-0.2425" z="-0.02"/>
   <gazebo>
-    <plugin filename="libignition-gazebo-mecanum-drive-system.so" name="ignition::gazebo::systems::MecanumDrive">
+    <plugin filename="gz-sim-mecanum-drive-system" name="gz::sim::systems::MecanumDrive">
+      <front_left_joint>front_left_wheel_joint</front_left_joint>
+      <front_right_joint>front_right_wheel_joint</front_right_joint>
+      <back_left_joint>rear_left_wheel_joint</back_left_joint>
+      <back_right_joint>rear_right_wheel_joint</back_right_joint>
+      <wheel_separation>0.485</wheel_separation>
+      <wheelbase>0.345</wheelbase>
+      <wheel_radius>${wheel_radius}</wheel_radius>
+      <odom_publish_frequency>50</odom_publish_frequency>
+      <frame_id>odom</frame_id>
       <child_frame_id>base_link</child_frame_id>
-      <wheel_separation>0.485</wheel_separation><wheelbase>0.345</wheelbase><wheel_radius>${wheel_radius}</wheel_radius>
     </plugin>
   </gazebo>

Commit message: refactor: improve simulation stability and sync navigation parameters

File: src/khr2026_team1_simulation/urdf/hand.xacro (robot description, xacro)
@@ -2,51 +2,65 @@
 <robot xmlns:xacro="http://www.ros.org/wiki/xacro">
   <xacro:macro name="robot_hand" params="base_link base_length base_width base_height">
-    <link name="lift_link">
-      <visual><origin xyz="0 0 0.15"/><geometry><box size="0.05 0.2 0.3"/></geometry><material name="grey"><color rgba="0.5 0.5 0.5 1.0"/></material></visual>
-      <collision><origin xyz="0 0 0.15"/><geometry><box size="0.05 0.2 0.3"/></geometry></collision>
-      <inertial><mass value="1.0"/><inertia ixx="0.01" ixy="0" ixz="0" iyy="0.01" iyz="0" izz="0.01"/></inertial>
-    </link>
-    <joint name="lift_joint" type="prismatic">
-      <parent link="${base_link}"/><child link="lift_link"/><origin xyz="${base_length/2 + 0.025} 0 ${base_height}"/><axis xyz="0 0 1"/><limit lower="0" upper="0.5" effort="100" velocity="0.5"/>
-    </joint>
-    <link name="gripper_base">
-      <visual><geometry><box size="0.1 0.2 0.05"/></geometry></visual>
-      <collision><geometry><box size="0.1 0.2 0.05"/></geometry></collision>
-      <inertial><mass value="0.2"/><inertia ixx="0.001" ixy="0" ixz="0" iyy="0.001" iyz="0" izz="0.001"/></inertial>
-    </link>
-    <joint name="gripper_base_joint" type="fixed">
-      <parent link="lift_link"/><child link="gripper_base"/><origin xyz="0.05 0 0.3"/>
-    </joint>
-    <link name="left_finger">
-      <visual><origin xyz="0.05 0 0"/><geometry><box size="0.1 0.02 0.05"/></geometry></visual>
-      <collision><origin xyz="0.05 0 0"/><geometry><box size="0.1 0.02 0.05"/></geometry></collision>
-      <inertial><mass value="0.1"/><inertia ixx="0.0001" ixy="0" ixz="0" iyy="0.0001" iyz="0" izz="0.0001"/></inertial>
-    </link>
-    <joint name="left_finger_joint" type="revolute">
-      <parent link="gripper_base"/><child link="left_finger"/><origin xyz="0.05 0.08 0"/><axis xyz="0 0 1"/><limit lower="-0.5" upper="0.5" effort="10" velocity="1.0"/>
-    </joint>
-    <link name="right_finger">
-      <visual><origin xyz="0.05 0 0"/><geometry><box size="0.1 0.02 0.05"/></geometry></visual>
-      <collision><origin xyz="0.05 0 0"/><geometry><box size="0.1 0.02 0.05"/></geometry></collision>
-      <inertial><mass value="0.1"/><inertia ixx="0.0001" ixy="0" ixz="0" iyy="0.0001" iyz="0" izz="0.0001"/></inertial>
-    </link>
-    <joint name="right_finger_joint" type="revolute">
-      <parent link="gripper_base"/><child link="right_finger"/><origin xyz="0.05 -0.08 0"/><axis xyz="0 0 1"/><limit lower="-0.5" upper="0.5" effort="10" velocity="1.0"/>
-    </joint>
-    <gazebo>
-      <plugin filename="libignition-gazebo-joint-state-publisher-system.so" name="ignition::gazebo::systems::JointStatePublisher"></plugin>
-      <plugin filename="libignition-gazebo-joint-position-controller-system.so" name="ignition::gazebo::systems::JointPositionController">
-        <joint_name>lift_joint</joint_name><p_gain>10000</p_gain>
-      </plugin>
-      <plugin filename="libignition-gazebo-joint-position-controller-system.so" name="ignition::gazebo::systems::JointPositionController">
-        <joint_name>left_finger_joint</joint_name><p_gain>100</p_gain>
-      </plugin>
-      <plugin filename="libignition-gazebo-joint-position-controller-system.so" name="ignition::gazebo::systems::JointPositionController">
-        <joint_name>right_finger_joint</joint_name><p_gain>100</p_gain>
-      </plugin>
-      <plugin filename="libignition-gazebo-pose-publisher-system.so" name="ignition::gazebo::systems::PosePublisher">
-        <publish_link_pose>true</publish_link_pose><use_pose_vector_msg>true</use_pose_vector_msg>
-      </plugin>
-    </gazebo>
+     <link name="lift_link">
+       <visual><origin xyz="0 0 0.15"/><geometry><box size="0.05 0.2 0.3"/></geometry><material name="grey"/></visual>
+       <collision><origin xyz="0 0 0.15"/><geometry><box size="0.05 0.2 0.3"/></geometry></collision>
+       <inertial><mass value="1.0"/><inertia ixx="0.01" ixy="0" ixz="0" iyy="0.01" iyz="0" izz="0.01"/></inertial>
+     </link>
+     <gazebo reference="lift_link">
+       <material>Gazebo/Grey</material>
+     </gazebo>
+     <joint name="lift_joint" type="prismatic">
+       <parent link="${base_link}"/><child link="lift_link"/><origin xyz="${base_length/2 + 0.025} 0 ${base_height}"/><axis xyz="0 0 1"/><limit lower="0" upper="0.5" effort="100" velocity="0.5"/>
+     </joint>
+     <link name="gripper_base">
+       <visual><geometry><box size="0.1 0.2 0.05"/></geometry><material name="grey"/></visual>
+       <collision><geometry><box size="0.1 0.2 0.05"/></geometry></collision>
+       <inertial><mass value="0.2"/><inertia ixx="0.001" ixy="0" ixz="0" iyy="0.001" iyz="0" izz="0.001"/></inertial>
+     </link>
+     <gazebo reference="gripper_base">
+       <material>Gazebo/Grey</material>
+     </gazebo>
+     <joint name="gripper_base_joint" type="fixed">
+       <parent link="lift_link"/><child link="gripper_base"/><origin xyz="0.05 0 0.3"/>
+     </joint>
+     <link name="left_finger">
+       <visual><origin xyz="0.05 0 0"/><geometry><box size="0.1 0.02 0.05"/></geometry><material name="black"/></visual>
+       <collision><origin xyz="0.05 0 0"/><geometry><box size="0.1 0.02 0.05"/></geometry></collision>
+       <inertial><mass value="0.1"/><inertia ixx="0.0001" ixy="0" ixz="0" iyy="0.0001" iyz="0" izz="0.0001"/></inertial>
+     </link>
+     <gazebo reference="left_finger">
+       <material>Gazebo/Black</material>
+     </gazebo>
+     <joint name="left_finger_joint" type="revolute">
+       <parent link="gripper_base"/><child link="left_finger"/><origin xyz="0.05 0.08 0"/><axis xyz="0 0 1"/><limit lower="-0.5" upper="0.5" effort="10" velocity="1.0"/>
+     </joint>
+     <link name="right_finger">
+       <visual><origin xyz="0.05 0 0"/><geometry><box size="0.1 0.02 0.05"/></geometry><material name="black"/></visual>
+       <collision><origin xyz="0.05 0 0"/><geometry><box size="0.1 0.02 0.05"/></geometry></collision>
+       <inertial><mass value="0.1"/><inertia ixx="0.0001" ixy="0" ixz="0" iyy="0.0001" iyz="0" izz="0.0001"/></inertial>
+     </link>
+     <gazebo reference="right_finger">
+       <material>Gazebo/Black</material>
+     </gazebo>
+     <joint name="right_finger_joint" type="revolute">
+       <parent link="gripper_base"/><child link="right_finger"/><origin xyz="0.05 -0.08 0"/><axis xyz="0 0 1"/><limit lower="-0.5" upper="0.5" effort="10" velocity="1.0"/>
+     </joint>
+     <gazebo>
+       <plugin filename="gz-sim-joint-state-publisher-system" name="gz::sim::systems::JointStatePublisher"></plugin>
+       <plugin filename="gz-sim-joint-position-controller-system" name="gz::sim::systems::JointPositionController">
+         <joint_name>lift_joint</joint_name><p_gain>10000</p_gain>
+       </plugin>
+       <plugin filename="gz-sim-joint-position-controller-system" name="gz::sim::systems::JointPositionController">
+         <joint_name>left_finger_joint</joint_name><p_gain>100</p_gain>
+       </plugin>
+       <plugin filename="gz-sim-joint-position-controller-system" name="gz::sim::systems::JointPositionController">
+         <joint_name>right_finger_joint</joint_name><p_gain>100</p_gain>
+       </plugin>
+        <!-- Removed to prevent conflict with Nav2/AMCL TF tree
+        <plugin filename="gz-sim-pose-publisher-system" name="gz::sim::systems::PosePublisher">
+          <publish_link_pose>true</publish_link_pose><use_pose_vector_msg>true</use_pose_vector_msg>
+        </plugin>
+        -->
+     </gazebo>
   </xacro:macro>
 </robot>

File: src/khr2026_team1_simulation/urdf/lidar.xacro (robot description, xacro)
@@ -6,5 +6,7 @@
       <visual>
         <geometry><cylinder radius="0.03" length="0.04"/></geometry>
-        <material name="black"/>
+        <material name="black">
+          <color rgba="0.1 0.1 0.1 1"/>
+        </material>
       </visual>
       <collision>
@@ -16,7 +18,8 @@
       <parent link="${parent_link}"/>
       <child link="laser_frame"/>
-      <origin xyz="0 0 0.2" rpy="0 0 0"/>
+      <origin xyz="-0.15 0 0.45" rpy="0 0 0"/>
     </joint>
     <gazebo reference="laser_frame">
+      <material>Gazebo/Black</material>
       <sensor name="lidar" type="gpu_lidar">
         <pose>0 0 0 0 0 0</pose>
@@ -29,5 +32,5 @@
           <scan>
             <horizontal>
-              <samples>360</samples>
+              <samples>720</samples>
               <resolution>1.0</resolution>
               <min_angle>-3.14159</min_angle>
@@ -36,5 +39,5 @@
           </scan>
           <range>
-            <min>0.12</min>
+            <min>0.15</min>
             <max>10.0</max>
             <resolution>0.01</resolution>

File: src/khr2026_team1_simulation/urdf/mecanum_wheel.xacro (robot description, xacro)
@@ -8,14 +8,27 @@
         <material name="black"><color rgba="0.1 0.1 0.1 1.0"/></material>
       </visual>
-      <collision>
-        <origin xyz="0 0 0" rpy="${pi/2} 0 0"/>
-        <geometry><cylinder radius="${radius}" length="${width}"/></geometry>
-      </collision>
-      <inertial>
-        <mass value="0.5"/>
-        <inertia ixx="0.001" ixy="0" ixz="0" iyy="0.001" iyz="0" izz="0.001"/>
-      </inertial>
-    </link>
-    <joint name="${prefix}_wheel_joint" type="continuous">
+       <collision>
+         <origin xyz="0 0 0" rpy="${pi/2} 0 0"/>
+         <geometry><cylinder radius="${radius}" length="${width}"/></geometry>
+         <surface>
+           <friction>
+             <ode>
+               <mu>1.0</mu>
+               <mu2>1.0</mu2>
+             </ode>
+           </friction>
+         </surface>
+       </collision>
+       <inertial>
+         <mass value="0.5"/>
+         <inertia ixx="0.001" ixy="0" ixz="0" iyy="0.001" iyz="0" izz="0.001"/>
+       </inertial>
+     </link>
+     <gazebo reference="${prefix}_wheel_link">
+       <material>Gazebo/Black</material>
+       <mu1>1.0</mu1>
+       <mu2>1.0</mu2>
+     </gazebo>
+     <joint name="${prefix}_wheel_joint" type="continuous">
       <parent link="base_link"/>
       <child link="${prefix}_wheel_link"/>
